File: pt4115/pt4115.kicad_pcb (KiCad board)
At the start: 2 copper layers, 30 x 11 mm, 10 parts, among them J1 DC IN, J2 LED, U1 PT4115

Commit message: Pcb updated
Parts:
- C1: value 100uF 35V -> 22uF 35V; footprint Capacitor_THT:CP_Radial_D5.0mm_P2.50mm -> Capacitor_Tantalum_SMD:CP_EIA-7343-31_Kemet-D
- moved R1 111.4 mm to (60.9, 43.9), turned to 90 degrees
- moved D1 110.0 mm to (55.7, 38.6)
- moved U1 109.7 mm to (55.8, 43.9)
- moved L1 109.0 mm to (48.2, 40.1)
- moved R2 108.9 mm to (62.8, 43.9), turned to 90 degrees
- moved J1 108.6 mm to (42.6, 38.0)
- moved R3 106.5 mm to (64.7, 43.9), turned to 90 degrees
- moved J2 106.3 mm to (71.0, 43.2)
- moved R4 104.1 mm to (66.5, 43.9), turned to 90 degrees
- moved C1 97.9 mm to (64.4, 38.9)
Routing:
- net Net-(C1-Pad2): track 14.0 -> 34.5 mm
- net Net-(C1-Pad1): track 28.1 -> 35.2 mm
- net Net-(D1-Pad2): track 23.4 -> 28.9 mm
- net Net-(J2-Pad1): track 17.6 -> 14.3 mm
- net Net-(L1-Pad1): track 6.71 -> 5.91 mm
- net Net-(J1-Pad3): track 12.9 -> 12.2 mm
Other:
- board size 30 x 11 mm -> 32.6 x 11 mm
- net class Default: trace_width 0.5 -> 0.7
