File: pt4115/pt4115.sch (KiCad schematic (older format))
At the start: 10 parts, among them J1 DC IN, J2 LED, U1 PT4115

Commit message: Pcb updated
Parts:
- C1: value 100uF 35V -> 22uF 35V; footprint Capacitor_THT:CP_Radial_D5.0mm_P2.50mm -> Capacitor_Tantalum_SMD:CP_EIA-7343-31_Kemet-D
Changed lines of the file:
@@
 EESchema Schematic File Version 4
+LIBS:pt4115-cache
 EELAYER 26 0
 EELAYER END
@@
 P 3200 4100
 F 0 "C1" H 3318 4146 50  0000 L CNN
-F 1 "100uF 35V" H 3318 4055 50  0000 L CNN
-F 2 "Capacitor_THT:CP_Radial_D5.0mm_P2.50mm" H 3238 3950 50  0001 C CNN
+F 1 "22uF 35V" H 3318 4055 50  0000 L CNN
+F 2 "Capacitor_Tantalum_SMD:CP_EIA-7343-31_Kemet-D" H 3238 3950 50  0001 C CNN
 F 3 "~" H 3200 4100 50  0001 C CNN
 	1    3200 4100
